File: buck_converter.kicad_sch (KiCad schematic)
At the start: 0 parts

Commit message: Buck converter sheet done
Parts:
- added C301: 0.1uF 10V, Capacitor_SMD:C_0603_1608Metric, symbol Device:C
- added C302, C303, C304: 22uF 10V, Capacitor_SMD:C_0805_2012Metric, symbol Device:C
- added C305: 1uF/10V, SparkFun-Capacitor:C_0603_1608Metric, symbol SparkFun-Capacitor:C_Small
- added D301: LED RED, LED_SMD:LED_0603_1608Metric, symbol Device:LED
- added D302: SMF5V0A, Diode_SMD:D_SMF, symbol Diode:SMF5V0A
- added L301: 2.2 uH/4.3A, Inductor_SMD:L_Sunlord_SWPA4020S, symbol Device:L
- added R301: 100k/1%, Resistor_SMD:R_01005_0402Metric, symbol Device:R
- added R302: 22.1k/1%, Resistor_SMD:R_01005_0402Metric, symbol Device:R
- added R303: 1k/1%, Resistor_SMD:R_01005_0402Metric, symbol Device:R
- added TP301, TP302: TestPoint, symbol Connector:TestPoint
- added U301: SY8253ADC, Package_TO_SOT_SMD:TSOT-23-6, symbol Regulator_Switching:LM2734X
Connections:
- new net: C303.2, R301.2, R302.1, U301.3 (FB)
- new net: C305.1, U301.1 (BOOST)
- new net: C305.2, L301.1, U301.6 (SW)
- new net: D301.2 (A), R303.2
- new net +3V3: C303.1, C304.1, L301.2, R301.1, R303.1, TP301.1
- new net GND: C301.2, C302.2, C304.2, D301.1 (K), D302.2 (A2), R302.2, U301.2 (GND)
- new net ORING_5V: C301.1, C302.1, D302.1 (A1), TP302.1, U301.4 (EN), U301.5 (VIN)
Other:
- note added: "Vout = 0.6(100+22.1)/22.1 = 3.31V"
