File: buck_converter.kicad_sch (KiCad schematic)
At the start: 14 parts, among them U301 SY8253ADC

Commit message: fin du schema et debut annotations precises
Other:
- note added: "Datasheet"
- note added: "Détail sur la diode"
- note added: "LDO ou Buck converter"
- note added: "visualisation de la puissance (on/off)"
