File: oring_power.kicad_sch (KiCad schematic)
At the start: 0 parts

Commit message: OR-ing sheet done
Parts:
- added C201: 1uF 10V, Capacitor_SMD:C_0603_1608Metric, symbol Device:C
- added R201, R202, R204: 100k/1%, Resistor_SMD:R_01005_0402Metric, symbol Device:R
- added R203, R205: 150k/1%, Resistor_SMD:R_01005_0402Metric, symbol Device:R
- added U201, U202: LM66100DCK, Package_TO_SOT_SMD:SOT-363_SC-70-6, symbol Power_Management:LM66100DCK
Connections:
- new net: R201.2, U201.5 (ST), U202.3 (~{CE})
- new net GND: C201.2, R203.2, R205.2, U201.2 (GND), U202.2 (GND)
- new net NOTIFY_3V3_CON1: R202.2, R203.1
- new net NOTIFY_3V3_CON2: R204.2, R205.1
- new net ORING_5V: C201.1, U201.6 (VOUT), U202.6 (VOUT)
- new net USBVDD_5V_CON1: R201.1, R202.1, U201.1 (VIN)
- new net USBVDD_5V_CON2: R204.1, U202.1 (VIN)
- no-connect marks 0 -> 1
Other:
- note added: "Follows reference design from LM66100 datasheet"

Commit message: Buck converter sheet done
Parts:
- added TP201, TP202: TestPoint, symbol Connector:TestPoint
Connections:
- net USBVDD_5V_CON1: now also TP201.1
- net USBVDD_5V_CON2: now also TP202.1
Changed lines of the file:
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@@
+	)
+	(junction
+		(at 130.81 106.68)
+		(diameter 0)
+		(color 0 0 0 0)
 	)
 	(junction
@@
 		(at 166.37 111.76)
 	)
-	(bus_entry
-		(at 147.32 146.05)
-		(size 2.54 2.54)
-		(stroke
-			(width 0)
-			(type default)
-		)
-	)
 	(wire
 		(pts
@@
 	(wire
 		(pts
+			(xy 130.81 106.68) (xy 151.13 106.68)
+		)
+		(stroke
+			(width 0)
+			(type default)
+		)
+	)
+	(wire
+		(pts
 			(xy 196.85 76.2) (xy 205.74 76.2)
 		)
@@
 	(wire
 		(pts
-			(xy 124.46 106.68) (xy 151.13 106.68)
+			(xy 124.46 106.68) (xy 130.81 106.68)
 		)
 		(stroke
@@
 	)
 	(symbol
+		(lib_id "Connector:TestPoint")
+		(at 130.81 106.68 0)
+		(unit 1)
+		(body_style 1)
+		(exclude_from_sim no)
+		(in_bom yes)
+		(on_board yes)
+		(in_pos_files yes)
+		(dnp no)
+		(fields_autoplaced yes)
+		(property "Reference" "TP202"
+			(at 133.35 102.1079 0)
+			(show_name no)
+			(do_not_autoplace no)
+			(effects
+				(font
+					(size 1.27 1.27)
+				)
+				(justify left)
+			)
+		)
+		(property "Value" "TestPoint"
+			(at 133.35 104.6479 0)
+			(show_name no)
+			(do_not_autoplace no)
+			(effects
+				(font
+					(size 1.27 1.27)
+				)
+				(justify left)
+			)
+		)
+		(property "Footprint" ""
+			(at 135.89 106.68 0)
+			(hide yes)
+			(show_name no)
+			(do_not_autoplace no)
+			(effects
+				(font
+					(size 1.27 1.27)
+				)
+			)
+		)
+		(property "Datasheet" ""
+			(at 135.89 106.68 0)
+			(hide yes)
+			(show_name no)
+			(do_not_autoplace no)
+			(effects
+				(font
+					(size 1.27 1.27)
+				)
+			)
+		)
+		(property "Description" "test point"
+			(at 130.81 106.68 0)
+			(hide yes)
+			(show_name no)
+			(do_not_autoplace no)
+			(effects
+				(font
+					(size 1.27 1.27)
+				)
+			)
+		)
+		(pin "1"
+		)
+		(instances
+			(project "USB-Thumb-Drive"
+				(path "/61284d1f-c8a6-45b4-aa7f-ae2816ab8ea5/c78825f3-dda6-4079-a5d7-5fb9e3395d2a"
+					(reference "TP202")
+					(unit 1)
+				)
+			)
+		)
+	)
+	(symbol
 		(lib_id "power:GND")
 		(at 115.57 97.79 0)
@@
 					(unit 1)
 				)
+			)
+		)
+	)
+	(symbol
+		(lib_id "Connector:TestPoint")
+		(at 134.62 76.2 0)
+		(unit 1)
+		(body_style 1)
+		(exclude_from_sim no)
+		(in_bom yes)
+		(on_board yes)
+		(in_pos_files yes)
+		(dnp no)
+		(fields_autoplaced yes)
+		(property "Reference" "TP201"
+			(at 137.16 71.6279 0)
+			(show_name no)
+			(do_not_autoplace no)
+			(effects
+				(font
+					(size 1.27 1.27)
+				)
+				(justify left)
+			)
+		)
+		(property "Value" "TestPoint"
+			(at 137.16 74.1679 0)
+			(show_name no)
+			(do_not_autoplace no)
+			(effects
+				(font
+					(size 1.27 1.27)
+				)
+				(justify left)
+			)
+		)
+		(property "Footprint" ""
+			(at 139.7 76.2 0)
+			(hide yes)
+			(show_name no)
+			(do_not_autoplace no)
+			(effects
+				(font
+					(size 1.27 1.27)
+				)
+			)
+		)
+		(property "Datasheet" ""
+			(at 139.7 76.2 0)
+			(hide yes)
+			(show_name no)
+			(do_not_autoplace no)
+			(effects
+				(font
+					(size 1.27 1.27)
+				)
+			)
+		)
+		(property "Description" "test point"
+			(at 134.62 76.2 0)
+			(hide yes)
+			(show_name no)
+			(do_not_autoplace no)
+			(effects
+				(font
+					(size 1.27 1.27)
+				)
+			)
+		)
+		(pin "1"
+		)
+		(instances
+			(project "USB-Thumb-Drive"
+				(path "/61284d1f-c8a6-45b4-aa7f-ae2816ab8ea5/c78825f3-dda6-4079-a5d7-5fb9e3395d2a"
+					(reference "TP201")
+					(unit 1)
+				)

Commit message: progress USB parts of the schematic
Changed lines of the file:
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@@
+	(wire
+		(pts
+			(xy 64.8462 67.3862) (xy 0.0762 67.3862)
+		)
+		(stroke
+			(width 0)
+			(type default)
+		)
+	)
 	(wire
 		(pts
@@
 	(wire
 		(pts
+			(xy 0.0762 67.3862) (xy 0.0762 0.0762)
+		)
+		(stroke
+			(width 0)
+			(type default)
+		)
+	)
+	(wire
+		(pts
 			(xy 115.57 76.2) (xy 124.46 76.2)
 		)
 		(stroke
+			(width 0)
+			(type default)
+		)
+	)
+	(wire
+		(pts
+			(xy 64.8462 45.7962) (xy 64.8462 67.3862)
+		)
+		(stroke
