File: oring_power.kicad_sch (KiCad schematic)
At the start: 10 parts, among them U201 LM66100DCK, U202 LM66100DCK

Commit message: Schema de l'eMMC et liaison au USB bridge
Changed lines of the file:
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@@
-	(wire
-		(pts
-			(xy 64.8462 67.3862) (xy 0.0762 67.3862)
-		)
-		(stroke
-			(width 0)
-			(type default)
-		)
-	)
 	(wire
 		(pts
@@
 		)
 		(stroke
-			(width 0)
-			(type default)
-		)
-	)
-	(wire
-		(pts
-			(xy 64.8462 45.7962) (xy 64.8462 67.3862)
-		)
-		(stroke

Commit message: fin du schema et debut annotations precises
Parts:
- removed C201: 1uF 10V, Capacitor_SMD:C_0603_1608Metric, symbol Device:C
- removed TP201, TP202: TestPoint, symbol Connector:TestPoint
Connections:
- net USBVDD_5V_CON2: now also U201.3 (~{CE})
Other:
- moved on the sheet: R201, R202, R203, R204, R205, U201, U202
