File: usb_bridge.kicad_sch (KiCad schematic)
At the start: 0 parts

Commit message: progress USB parts of the schematic
Parts:
- added C401: 2.2nF/100V, SparkFun-Capacitor:C_0603_1608Metric, symbol SparkFun-Capacitor:C_Small
- added C402: 100nF/10V, SparkFun-Capacitor:C_0603_1608Metric, symbol SparkFun-Capacitor:C_Small
- added C403, C404, C405, C406: 0.1uF/10V, SparkFun-Capacitor:C_0603_1608Metric, symbol SparkFun-Capacitor:C_Small
- added C407: 4.7uF/10V, SparkFun-Capacitor:C_0603_1608Metric, symbol SparkFun-Capacitor:C_Small
- added C408, C409: 1uF/10V, SparkFun-Capacitor:C_0603_1608Metric, symbol SparkFun-Capacitor:C_Small
- added D401: LED RED, LED_SMD:LED_0603_1608Metric, symbol Device:LED
- added R401, R402, R404, R405, R406: 10k/1%, Resistor_SMD:R_01005_0402Metric, symbol Device:R
- added R403: 330/1%, Resistor_SMD:R_01005_0402Metric, symbol Device:R
- added U401: USB2244-AEZG-06, footprints:QFN36_6X6MC_MCH, symbol ul_USB2244:USB2244-AEZG-06
- added U402: AT24CS04-STUM, Package_TO_SOT_SMD:SOT-23-5, symbol Memory_EEPROM:AT24CS04-STUM
- added U403: D3V3XA4B10LP, Package_DFN_QFN:Diodes_UDFN-10_1x2.5mm_P0.5mm, symbol Power_Protection:D3V3XA4B10LP
- added Y401: SG-210STF, Oscillator:Oscillator_SMD_SeikoEpson_SG210-4Pin_2.5x2.0mm, symbol Oscillator:SG-210STF
Connections:
- new net: R404.2, U401.26 (SD_NCD)
- new net: C409.1, U401.34 (VDD18PLL)
- new net: C408.2, U401.13 (VDD18)
- new net: C401.1, R401.1, U401.18 (RESET_N)
- new net: D401.1 (K), R403.1
- new net: D401.2 (A), U401.1 (LED)
- new net: R402.2, U401.35 (RBIAS)
- new net: U401.33 (XTAL1(CLKIN)), Y401.3 (OUT)
- new net +3V3: C402.1, C403.1, C404.1, C405.1, C406.1, C407.1, R401.2, R405.1, R406.1, U401.14 (VDD33), U401.22 (VDD33), U401.36 (VDDA33), U401.6 (VDD33), U402.4 (VCC), Y401.1 (~{ST}), Y401.4 (Vcc)
- new net GND: C401.2, C402.2, C403.2, C404.2, C405.2, C406.2, C407.2, C408.1, C409.2, R402.1, R403.2, R404.1, U401.28 (TEST), U401.37 (EPAD), U402.2 (GND), U402.5 (WP), U403.3 (VSS), U403.8 (VSS), Y401.2 (GND)
- new net SCK_USB2244: R406.2, U401.31 (TXD/SCK), U402.1 (SCL)
- new net SDA_USB2244: R405.2, U401.27 (RXD/SDA), U402.3 (SDA)
- new net STORAGE_USB+: U401.2 (USB+), U403.1
- new net STORAGE_USB-: U401.3 (USB-), U403.2
- no-connect marks 0 -> 4
Other:
- note added: "Decoupling capacitors input power"
- note added: "ESD protection"
