File: usb_bridge.kicad_sch (KiCad schematic)
At the start: 20 parts, among them U401 USB2244-AEZG-06, U402 AT24CS04-STUM, U403 D3V3XA4B10LP, Y401 SG-210STF

Commit message: Schema de l'eMMC et liaison au USB bridge
Parts:
- added R407, R408, R409, R410, R411, R412, R413, R414: 0 Ohm, Resistor_SMD:R_01005_0402Metric, symbol Device:R
Connections:
- net SD_D5: now reaches U401.10 (SD_D5)
- net SD_D5: now also R412.2
- net MMC_CMD: now reaches U401.11 (SD_CMD)
- net SD_D4: now reaches U401.20 (SD_D4)
- net SD_D4: now also R411.2
- net SD_D3: now reaches U401.23 (SD_D3)
- net SD_D3: now also R410.2
- net SD_D2: now reaches U401.25 (SD_D2)
- net SD_D2: now also R409.2
- net SD_D1: now reaches U401.4 (SD_D1)
- net SD_D1: now also R408.2
- net SD_D0: now reaches U401.5 (SD_D0)
- net SD_D0: now also R407.2
- net SD_D7: now reaches U401.7 (SD_D7)
- net SD_D7: now also R414.2
- net SD_D6: now reaches U401.8 (SD_D6)
- net SD_D6: now also R413.2
- net MMC_CLK: now reaches U401.9 (SD_CLK)
Other:
- note removed: "Decoupling capacitors input power"
- moved on the sheet: C402, C403, C404, C405, C406, C407, R405, R406, U402

Commit message: avancees majeures sur le schema
Connections:
- no-connect marks 4 -> 8
Changed lines of the file:
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@@
+	)
+	(no_connect
+		(at 236.22 25.4)
 	)
 	(no_connect
 		(at 153.67 74.93)
+	)
+	(no_connect
+		(at 210.82 25.4)
 	)
 	(no_connect
@@
 	)
 	(no_connect
+		(at 210.82 40.64)
+	)
+	(no_connect
 		(at 153.67 102.87)
 	)
+	(no_connect
+		(at 236.22 40.64)
+	)
 	(bus_entry

Commit message: fin du schema et debut annotations precises
Connections:
- net GND: now also U401.30 (SD_WP)
- net MMCD0: now reaches R407.1
- net MMCD1: now reaches R408.1
- net MMCD2: now reaches R409.1
- net MMCD5: now reaches R412.1
- net MMCD6: now reaches R413.1
- net MMCD7: now reaches R414.1
- net MMCD4: now reaches R411.1
- net MMCD3: now reaches R410.1
Other:
- moved on the sheet: R407, R408, R409, R410, R411, R412, R413, R414

Commit message: fin des annotations, schema terminé
Other:
- note added: "*1"
- note added: "*2"
- note added: "*3"
- note added: "Decoupling capacitor"
- note added: "EEPROM Memory"
- note added: "External clock"
- note added: "decoupling capacitor"
- moved on the sheet: C401, C402, C403, C404, C405, C406, C407, C408, C409, D401, R401, R402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
