File: rp2040.kicad_sch (KiCad schematic)
At the start: 0 parts

Commit message: Progress RP2040 schematic
Parts:
- added C502, C503: 15pF/10V, SparkFun-Capacitor:C_0603_1608Metric, symbol SparkFun-Capacitor:C_Small
- added R502, R503: 10k/1%, Resistor_SMD:R_01005_0402Metric, symbol Device:R
- added R504: 1k/1%, Resistor_SMD:R_01005_0402Metric, symbol Device:R
- added U501: RP2040, Package_DFN_QFN:QFN-56-1EP_7x7mm_P0.4mm_EP3.2x3.2mm, symbol MCU_RaspberryPi:RP2040
- added U503: D3V3XA4B10LP, Package_DFN_QFN:Diodes_UDFN-10_1x2.5mm_P0.5mm, symbol Power_Protection:D3V3XA4B10LP
- added Y501: Crystal_GND24, Crystal:Crystal_SMD_3225-4Pin_3.2x2.5mm, symbol Device:Crystal_GND24
Connections:
- new net: R504.1, U501.21 (XOUT)
- new net: C503.2, R504.2, Y501.3
- new net: C502.2, U501.20 (XIN), Y501.1
- new net: R503.1, U501.47 (USB_DP)
- new net: R502.1, U501.46 (USB_DM)
- new net: U501.1 (IOVDD), U501.10 (IOVDD), U501.22 (IOVDD), U501.33 (IOVDD), U501.42 (IOVDD), U501.49 (IOVDD)
- new net: U501.23 (DVDD), U501.50 (DVDD)
- new net GND: C502.1, C503.1, U503.3 (VSS), U503.8 (VSS), Y501.2 (G), Y501.4 (G)
- new net RP_USB_D+: R502.2, U503.1
- new net RP_USB_D-: R503.2, U503.2
