File: rp2040.kicad_sch (KiCad schematic)
At the start: 8 parts, among them U501 RP2040, U503 D3V3XA4B10LP, Y501 Crystal_GND24

Commit message: avancees majeures sur le schema
Parts:
- removed C502, C503: 15pF/10V, SparkFun-Capacitor:C_0603_1608Metric, symbol SparkFun-Capacitor:C_Small
- removed U503: D3V3XA4B10LP, Package_DFN_QFN:Diodes_UDFN-10_1x2.5mm_P0.5mm, symbol Power_Protection:D3V3XA4B10LP
- removed Y501: Crystal_GND24, Crystal:Crystal_SMD_3225-4Pin_3.2x2.5mm, symbol Device:Crystal_GND24
- added C501, C520: 1u, Capacitor_SMD:C_0402_1005Metric, symbol Device:C
- added C502: 10u, Capacitor_SMD:C_0805_2012Metric, symbol Device:C
- added C504, C505, C506, C507, C522: 100n, Capacitor_SMD:C_0402_1005Metric, symbol Device:C
- added C521, C523: 15pF/10V, SparkFun-Capacitor:C_0603_1608Metric, symbol SparkFun-Capacitor:C_Small
- added J501: Conn_01x02, Connector_PinHeader_2.54mm:PinHeader_1x02_P2.54mm_Vertical, symbol Connector_Generic:Conn_01x02
- added R501: 1k, Resistor_SMD:R_0402_1005Metric, symbol Device:R
- added R505: DNF, Resistor_SMD:R_0402_1005Metric, symbol Device:R
- added R506: 1k/1%, Resistor_SMD:R_01005_0402Metric, symbol Device:R
- added R507, R508: 4.7k/1%, Resistor_SMD:R_01005_0402Metric, symbol Device:R
- added R509: 10k/1%, Resistor_SMD:R_01005_0402Metric, symbol Device:R
- added U502: W25Q128JVS, Package_SO:SOIC-8_5.3x5.3mm_P1.27mm, symbol Memory_Flash:W25Q128JVS
- added U504: D3V3XA4B10LP, Package_DFN_QFN:Diodes_UDFN-10_1x2.5mm_P0.5mm, symbol Power_Protection:D3V3XA4B10LP
- added Y502: Crystal_GND24, Crystal:Crystal_SMD_3225-4Pin_3.2x2.5mm, symbol Device:Crystal_GND24
- R502, R503: value 10k/1% -> 4.7k/1%
- R504: value 1k/1% -> 10k/1%
Connections:
- net GND: now also U501.19 (TESTEN), U501.57 (GND), C501.2, C502.2, C504.2, C505.2, C506.2, C507.2, C520.2, C521.1, C522.2, C523.1, J501.2 (Pin_2), U502.4 (GND), U504.3 (VSS), U504.8 (VSS), Y502.2 (G), Y502.4 (G)
- net RP_USB_D+: now also R504.2, U501.47 (USB_DP), U504.1; no longer R502.2
- net RP_USB_D-: now also U501.46 (USB_DM), R509.2, U504.2; no longer R503.2
- net RP_XOUT: now reaches U501.21 (XOUT)
- net RP_XOUT: now also R506.1; no longer R504.1
- net RP_XIN: now reaches U501.20 (XIN)
- net RP_XIN: now also C521.2, Y502.1
- net I2C0_SDA: now reaches R503.1
- net I2C0_SDA: now also U501.6 (GPIO4); no longer U501.47 (USB_DP)
- net I2C_SCL: now reaches R502.1
- net I2C_SCL: now also U501.5 (GPIO3); no longer U501.46 (USB_DM)
- net +3V3: now reaches U501.1 (IOVDD), U501.10 (IOVDD), U501.22 (IOVDD), U501.33 (IOVDD), U501.42 (IOVDD), U501.49 (IOVDD)
- net +3V3: now also R502.2, R503.2, U501.43 (ADC_AVDD), U501.44 (VREG_VIN), U501.48 (USB_VDD), C501.1, C502.1, C504.1, C505.1, C506.1, C507.1, R505.1, R507.2, R508.2, U502.8 (VCC)
- net SPI_CLK: now reaches U501.13 (GPIO10)
- net SPI_MOSI: now reaches U501.14 (GPIO11)
- net SPI_MISO: now reaches U501.15 (GPIO12)
- net SPI_CS: now reaches U501.16 (GPIO13)
- net GPIO14: now reaches U501.17 (GPIO14)
- net GPIO15: now reaches U501.18 (GPIO15)
- net UART_TX: now reaches U501.2 (GPIO0)
- net +1V1: now reaches U501.23 (DVDD), U501.50 (DVDD)
- net +1V1: now also U501.45 (VREG_VOUT), C520.1, C522.1
- net SWCLK: now reaches U501.24 (SWCLK)
- net SWDIO: now reaches U501.25 (SWDIO)
- net RUN: now reaches U501.26 (RUN)
- net LED_A: now reaches U501.27 (GPIO16)
- net LED_B: now reaches U501.28 (GPIO17)
- net LED_C: now reaches U501.29 (GPIO18)
- net UART_RX: now reaches U501.3 (GPIO1)
- net GPIO24: now reaches U501.36 (GPIO24)
- net GPIO25: now reaches U501.37 (GPIO25)
- net I2C_SDA: now reaches U501.4 (GPIO2)
- net I2C_SDA: now also R508.1
- net QSPI_SD3: now reaches U501.51 (QSPI_SD3)
- net QSPI_SD3: now also U502.7 (~{HOLD}/~{RESET}/IO_{3})
- net QSPI_SCLK: now reaches U501.52 (QSPI_SCLK)
- net QSPI_SCLK: now also U502.6 (CLK)
- net QSPI_SD0: now reaches U501.53 (QSPI_SD0)
- net QSPI_SD0: now also U502.5 (DI/IO_{0})
- net QSPI_SD2: now reaches U501.54 (QSPI_SD2)
- net QSPI_SD2: now also U502.3 (~{WP}/IO_{2})
- net QSPI_SD1: now reaches U501.55 (QSPI_SD1)
- net QSPI_SD1: now also U502.2 (DO/IO_{1})
- net QSPI_SS: now reaches U501.56 (~{QSPI_SS})
- net QSPI_SS: now also R501.1, R505.2, U502.1 (~{CS})
- net I2C0_SCL: now reaches U501.7 (GPIO5)
- net I2C0_SCL: now also R507.1
- new net: C523.2, R506.2, Y502.3
- new net USB_D+: R504.1
- new net USB_D-: R509.1
- new net ~{USB_BOOT}: J501.1 (Pin_1), R501.2
- no-connect marks 0 -> 18
Other:
- added sheet GPIO breakouts (gpio.kicad_sch)
- added sheet Sensors and OLED (sensors.kicad_sch)
- note added: "ESD protection on USB D+ and D-"
- note added: "Flash sub circuit"
- note added: "Make sure C501 is close to pin 44 of RP2040"
- note added: "Make sure C520 is close to pin 45 of RP2040"
- moved on the sheet: U501

Commit message: fin du schema et debut annotations precises
Connections:
- net USB_D+ is gone; now on net RP_USB_D-: R504.1
- net USB_D- is gone; now on net RP_USB_D+: R509.1
- net RP_USB_D+: no longer R504.2, U501.47 (USB_DP)
- net RP_USB_D-: no longer R509.2, U501.46 (USB_DM)
- new net: R504.2, U501.46 (USB_DM)
- new net: R509.2, U501.47 (USB_DP)
- no-connect marks 18 -> 19
Other:
- note added: "Crystal"
- note added: "Decoupling capacitor"
- note added: "GPIO Breakouts"
- note added: "L'objectif est de pouvoir relier des pins du microcontrolleur à des composants externes à la carte (par exemple d'autres capteurs). Pour assurer une adaptabilité max, les pins sont destinés à plusieurs protocoles (SPI, I2C et UART). Il y a aussi des GPIO du MCU qui vont vers des LEDs pour donner des possibilités d'affichage."
- note added: "Pull up resistors for I2C signals"
- moved on the sheet: C501, C502, C504, C505, C506, C507, C520, C521, C522, C523, J501, R501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
