File: USB-Thumb-Drive.kicad_sch (KiCad schematic)
At the start: 10 parts, among them J101 USB_C_Receptacle_USB2.0_14P, J102 USB_C_Receptacle_USB2.0_14P

Commit message: Schema de l'eMMC et liaison au USB bridge
Other:
- sheet USB_BRIDGE ports: added MMCD[0:7], MMC_CLK, MMC_CMD; removed none
- sheet eMMC_STORAGE ports: added MMC_CLK, MMC_CMD, MMC_DATA[0:7]; removed none
Changed lines of the file:
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@@
+	(wire
+		(pts
+			(xy 222.25 93.98) (xy 222.25 96.52)
+		)
+		(stroke
+			(width 0)
+			(type default)
+		)
+	)
 	(wire
 		(pts
@@
 	(wire
 		(pts
+			(xy 214.63 93.98) (xy 222.25 93.98)
+		)
+		(stroke
+			(width 0)
+			(type default)
+		)
+	)
+	(wire
+		(pts
 			(xy 68.58 132.08) (xy 90.17 132.08)
 		)
@@
 	(wire
 		(pts
+			(xy 222.25 96.52) (xy 228.6 96.52)
+		)
+		(stroke
+			(width 0)
+			(type default)
+		)
+	)
+	(wire
+		(pts
 			(xy 80.01 109.22) (xy 80.01 44.45)
 		)
@@
 	(wire
 		(pts
+			(xy 214.63 87.63) (xy 228.6 87.63)
+		)
+		(stroke
+			(width 0)
+			(type default)
+		)
+	)
+	(wire
+		(pts
 			(xy 66.04 31.75) (xy 68.58 31.75)
 		)
@@
 		(pts
 			(xy 36.83 73.66) (xy 36.83 76.2)
+		)
+		(stroke
+			(width 0)
+			(type default)
+		)
+	)
+	(wire
+		(pts
+			(xy 214.63 85.09) (xy 228.6 85.09)
 		)
 		(stroke
@@
 			)
 		)
+		(pin "MMCD[0:7]" bidirectional
+			(at 214.63 93.98 0)
+			(effects
+				(font
+					(size 1.27 1.27)
+				)
+				(justify right)
+			)
+		)
+		(pin "MMC_CLK" output
+			(at 214.63 85.09 0)
+			(effects
+				(font
+					(size 1.27 1.27)
+				)
+				(justify right)
+			)
+		)
+		(pin "MMC_CMD" bidirectional
+			(at 214.63 87.63 0)
+			(effects
+				(font
+					(size 1.27 1.27)
+				)
+				(justify right)
+			)
+		)
 		(instances
 			(project "USB-Thumb-Drive"
@@
 			)
 		)
+		(pin "MMC_CLK" input
+			(at 228.6 85.09 180)
+			(effects
+				(font
+					(size 1.27 1.27)
+				)
+				(justify left)
+			)
+		)
+		(pin "MMC_CMD" bidirectional
+			(at 228.6 87.63 180)
+			(effects
+				(font
+					(size 1.27 1.27)
+				)
+				(justify left)
+			)
+		)
+		(pin "MMC_DATA[0:7]" bidirectional
+			(at 228.6 96.52 180)
+			(effects
+				(font
+					(size 1.27 1.27)
+				)
+				(justify left)
+			)
+		)

Commit message: avancees majeures sur le schema
Parts:
- added R107: 2m/1%, Resistor_SMD:R_01005_0402Metric, symbol Device:R
- added R108: 2m, Resistor_SMD:R_01005_0402Metric, symbol Device:R
- added U101: D3V3XA4B10LP, Package_DFN_QFN:Diodes_UDFN-10_1x2.5mm_P0.5mm, symbol Power_Protection:D3V3XA4B10LP
Connections:
- net GND: now also U101.3 (VSS), U101.8 (VSS)
- net USB_CC1_CON1: now reaches J101.A5 (CC1), R102.1
- net USB_CC1_CON1: now also U101.1
- net USB_CC2_CON1: now reaches J101.B5 (CC2), R103.1
- net USB_CC2_CON1: now also U101.2
- net USB_CC1_CON2: now reaches J102.A5 (CC1), R105.1
- net USB_CC1_CON2: now also U101.4
- net USB_CC2_CON2: now reaches J102.B5 (CC2), R106.1
- net USB_CC2_CON2: now also U101.5
- net ORING_POWER/USBVDD_5V_CON1 renamed VBUS_STORAGE
- net VBUS_STORAGE: now also R108.1
- net ORING_POWER/USBVDD_5V_CON2 renamed VBUS_MCU
- net VBUS_MCU: now also R107.1
- new net VBUS_MCU_IN-: R107.2
- new net VBUS_STORAGE_IN-: R108.2
- no-connect marks 0 -> 4
Other:
- sheet RP2040 ports: added CON1_ROOT_IN+, CON1_ROOT_IN-, CON2_ROOT_IN+, CON2_ROOT_IN-, GPIO24, GPIO25; removed none
- moved on the sheet: R102, R103, R105, R106

Commit message: fin du schema et debut annotations precises
Parts:
- added H101, H102, H103, H104: MountingHole, MountingHole:MountingHole_2.2mm_M2, symbol Mechanical:MountingHole
- added TP101, TP102: TestPoint, symbol Connector:TestPoint
Connections:
- net VBUS_MCU_IN-: now also TP102.1
- net VBUS_STORAGE: now also TP101.1
Other:
- sheet USB_BRIDGE ports: added MMCD[0..7]; removed MMCD[0:7]
- sheet eMMC_STORAGE ports: added MMCDA[0..7]; removed MMC_DATA[0:7]
- moved on the sheet: C101, C102, J101, J102, R101, R102, R103, R104, R105, R106, R107, U101
