File: gpio.kicad_sch (KiCad schematic)
At the start: 8 parts, among them J801 Conn_01x03, J802 Conn_01x12

Commit message: fin du schema et debut annotations precises
Other:
- moved on the sheet: D801, D802, D803, J801, J802, R801, R802, R803
