File: emmc_storage.kicad_sch (KiCad schematic)
At the start: 0 parts

Commit message: Schema de l'eMMC et liaison au USB bridge
Parts:
- added C601, C602, C604: 0.1uF/10V, SparkFun-Capacitor:C_0603_1608Metric, symbol SparkFun-Capacitor:C_Small
- added C603, C605: 2.2uF/10V, SparkFun-Capacitor:C_0603_1608Metric, symbol SparkFun-Capacitor:C_Small
- added C606: 1uF/10V, SparkFun-Capacitor:C_0603_1608Metric, symbol SparkFun-Capacitor:C_Small
- added FB601: FerriteBead, Inductor_SMD:L_Panasonic_PCC-M0530M, symbol Device:FerriteBead
- added NT602: NetTie_3, symbol Device:NetTie_3
- added R601, R602, R603, R604, R605, R606, R607, R608: 47k/1%, Resistor_SMD:R_01005_0402Metric, symbol Device:R
- added R609: 22/1%, Resistor_SMD:R_01005_0402Metric, symbol Device:R
- added R610, R611: 10k/1%, Resistor_SMD:R_01005_0402Metric, symbol Device:R
- added U601: MTFC64GAPALBH-IT, MTFC64GAPALBH-IT:BGA153N50P14X14_1300X1150X110N, symbol MTFC64GAPALBH-IT:MTFC64GAPALBH-IT
Connections:
- new net: R611.1, U601.K5 (RST_N)
- new net: U601.A1 (NC), U601.A10 (NC), U601.A11 (NC), U601.A12 (NC), U601.A13 (NC), U601.A14 (NC), U601.A2 (NC), U601.A8 (NC), U601.A9 (NC), U601.B1 (NC), U601.B10 (NC), U601.B11 (NC), U601.B12 (NC), U601.B13 (NC), U601.B14 (NC), U601.B7 (NC), U601.B8 (NC), U601.B9 (NC), U601.C1 (NC), U601.C10 (NC), U601.C11 (NC), U601.C12 (NC), U601.C13 (NC), U601.C14 (NC), U601.C3 (NC), U601.C5 (NC), U601.C7 (NC), U601.C8 (NC), U601.C9 (NC), U601.D1 (NC), U601.D12 (NC), U601.D13 (NC), U601.D14 (NC), U601.D2 (NC), U601.D3 (NC), U601.D4 (NC), U601.E1 (NC), U601.E12 (NC), U601.E13 (NC), U601.E14 (NC), U601.E2 (NC), U601.E3 (NC), U601.F1 (NC), U601.F12 (NC), U601.F13 (NC), U601.F14 (NC), U601.F2 (NC), U601.F3 (NC), U601.G1 (NC), U601.G12 (NC), U601.G13 (NC), U601.G14 (NC), U601.G2 (NC), U601.G3 (NC), U601.H1 (NC), U601.H12 (NC), U601.H13 (NC), U601.H14 (NC), U601.H2 (NC), U601.H3 (NC), U601.J1 (NC), U601.J12 (NC), U601.J13 (NC), U601.J14 (NC), U601.J2 (NC), U601.J3 (NC), U601.K1 (NC), U601.K12 (NC), U601.K13 (NC), U601.K14 (NC), U601.K2 (NC), U601.K3 (NC), U601.L1 (NC), U601.L12 (NC), U601.L13 (NC), U601.L14 (NC), U601.L2 (NC), U601.L3 (NC), U601.M1 (NC), U601.M10 (NC), U601.M11 (NC), U601.M12 (NC), U601.M13 (NC), U601.M14 (NC), U601.M2 (NC), U601.M3 (NC), U601.M7 (NC), U601.M8 (NC), U601.M9 (NC), U601.N1 (NC), U601.N10 (NC), U601.N11 (NC), U601.N12 (NC), U601.N13 (NC), U601.N14 (NC), U601.N3 (NC), U601.N6 (NC), U601.N7 (NC), U601.N8 (NC), U601.N9 (NC), U601.P1 (NC), U601.P11 (NC), U601.P12 (NC), U601.P13 (NC), U601.P14 (NC), U601.P2 (NC), U601.P7 (NC), U601.P8 (NC), U601.P9 (NC)
- new net: U601.A7 (RFU), U601.E5 (RFU), U601.K6 (RFU), U601.K7 (RFU)
- new net: R609.1, U601.M6 (CLK)
- new net +3V3: FB601.2, R611.2
- new net GND: C601.2, C602.2, C603.2, C604.2, C605.2, C606.2, U601.A6 (VSS), U601.C4 (VSSQ), U601.E7 (VSS), U601.G5 (VSS), U601.H10 (VSS), U601.J5 (VSS), U601.K8 (VSS), U601.N2 (VSSQ), U601.N5 (VSSQ), U601.P4 (VSSQ), U601.P6 (VSSQ)
- new net MMCDA0: R601.2, U601.A3 (DAT0)
- new net MMCDA1: R602.2, U601.A4 (DAT1)
- new net MMCDA2: R603.2, U601.A5 (DAT2)
- new net MMCDA3: R604.2, U601.B2 (DAT3)
- new net MMCDA4: R605.2, U601.B3 (DAT4)
- new net MMCDA5: R606.2, U601.B4 (DAT5)
- new net MMCDA6: R607.2, U601.B5 (DAT6)
- new net MMCDA7: R608.2, U601.B6 (DAT7)
- new net MMC_CLK: R609.2
- new net MMC_CMD: R610.2, U601.M5 (CMD)
- new net VCC: C601.1, C605.1, FB601.1, NT602.2, U601.E6 (VCC), U601.F5 (VCC), U601.J10 (VCC), U601.K9 (VCC)
- new net VCCQ: C602.1, C603.1, NT602.1, R601.1, R602.1, R603.1, R604.1, R605.1, R606.1, R607.1, R608.1, R610.1, U601.C6 (VCCQ), U601.M4 (VCCQ), U601.N4 (VCCQ), U601.P3 (VCCQ), U601.P5 (VCCQ)
- new net Vddim_eMMC: C604.1, C606.1, NT602.3, U601.C2 (VDDIM)

Commit message: avancees majeures sur le schema
Parts:
- removed NT602: NetTie_3, symbol Device:NetTie_3
- added NT601: NetTie_3, symbol Device:NetTie_3
Connections:
- net VCC: now also NT601.2
- net VCCQ: now also NT601.1
- net Vddim_eMMC: now also NT601.3
Changed lines of the file:
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@@
 	(wire
 		(pts
-			(xy 200.66 66.04) (xy 231.14 66.04)
-		)
-		(stroke
-			(width 0)
-			(type default)
-		)
-	)
-	(wire
-		(pts
 			(xy 269.24 76.2) (xy 269.24 77.47)
 		)
@@
 	(wire
 		(pts
-			(xy 179.07 66.04) (xy 200.66 66.04)
+			(xy 179.07 66.04) (xy 231.14 66.04)
 		)
 		(stroke
@@
 		)
 	)
-	(label "Vcc_eMMC"
-		(at 179.07 38.1 0)
-		(effects
-			(font
-				(size 1.27 1.27)
-			)
-			(justify left bottom)
-		)
-	)
 	(label "Vccq_eMMC"
 		(at 80.01 48.26 0)
@@
 		)
 	)
-	(label "MMCDA6"
-		(at 111.76 101.6 0)
+	(label "Vcc_eMMC"
+		(at 182.88 38.1 0)
 		(effects
 			(font
@@
 		)
 	)
-	(label "Vccq_eMMC"
-		(at 185.42 66.04 0)
+	(label "MMCDA6"
+		(at 111.76 101.6 0)
 		(effects
 			(font
@@
 		)
 	)
+	(label "Vccq_eMMC"
+		(at 185.42 66.04 0)
+		(effects
+			(font
+				(size 1.27 1.27)
+			)
+			(justify left bottom)
+		)
+	)
 	(label "MMCDA5"
 		(at 111.76 99.06 0)
@@
 	)
 	(symbol
+		(lib_id "Device:NetTie_3")
+		(at 242.57 43.18 90)
+		(unit 1)
+		(body_style 1)
+		(exclude_from_sim no)
+		(in_bom no)
+		(on_board yes)
+		(in_pos_files yes)
+		(dnp no)
+		(fields_autoplaced yes)
+		(property "Reference" "NT601"
+			(at 246.38 41.9099 90)
+			(show_name no)
+			(do_not_autoplace no)
+			(effects
+				(font
+					(size 1.27 1.27)
+				)
+				(justify right)
+			)
+		)
+		(property "Value" "NetTie_3"
+			(at 246.38 44.4499 90)
+			(show_name no)
+			(do_not_autoplace no)
+			(effects
+				(font
+					(size 1.27 1.27)
+				)
+				(justify right)
+			)
+		)
+		(property "Footprint" ""
+			(at 242.57 43.18 0)
+			(hide yes)
+			(show_name no)
+			(do_not_autoplace no)
+			(effects
+				(font
+					(size 1.27 1.27)
+				)
+			)
+		)
+		(property "Datasheet" ""
+			(at 242.57 43.18 0)
+			(hide yes)
+			(show_name no)
+			(do_not_autoplace no)
+			(effects
+				(font
+					(size 1.27 1.27)
+				)
+			)
+		)
+		(property "Description" "Net tie, 3 pins"
+			(at 242.57 43.18 0)
+			(hide yes)
+			(show_name no)
+			(do_not_autoplace no)
+			(effects
+				(font
+					(size 1.27 1.27)
+				)
+			)
+		)
+		(pin "1"
+		)
+		(pin "3"
+		)
+		(pin "2"
+		)
+		(instances
+			(project "USB-Thumb-Drive"
+				(path "/61284d1f-c8a6-45b4-aa7f-ae2816ab8ea5/ca50ca8d-e0c7-4aad-ae92-c1fe4b50bba9"
+					(reference "NT601")
+					(unit 1)
+				)
+			)
+		)
+	)
+	(symbol
 		(lib_id "power:PWR_FLAG")
 		(at 200.66 38.1 0)
@@
 					(unit 1)
 				)
-			)
-		)
-	)
-	(symbol
-		(lib_id "Device:NetTie_3")
-		(at 242.57 43.18 90)
-		(unit 1)
-		(body_style 1)
-		(exclude_from_sim no)
-		(in_bom no)
-		(on_board yes)
-		(in_pos_files yes)
-		(dnp no)
-		(fields_autoplaced yes)
-		(property "Reference" "NT602"
-			(at 246.38 41.9099 90)
-			(show_name no)
-			(do_not_autoplace no)
-			(effects
-				(font
-					(size 1.27 1.27)
-				)
-				(justify right)
-			)
-		)
-		(property "Value" "NetTie_3"
-			(at 246.38 44.4499 90)
-			(show_name no)
-			(do_not_autoplace no)
-			(effects
-				(font
-					(size 1.27 1.27)
-				)
-				(justify right)
-			)
-		)
-		(property "Footprint" ""
-			(at 242.57 43.18 0)
-			(hide yes)
-			(show_name no)
-			(do_not_autoplace no)
-			(effects
-				(font
-					(size 1.27 1.27)
-				)
-			)
-		)
-		(property "Datasheet" ""
-			(at 242.57 43.18 0)
-			(hide yes)
-			(show_name no)
-			(do_not_autoplace no)
-			(effects
-				(font
-					(size 1.27 1.27)
-				)
-			)
-		)
-		(property "Description" "Net tie, 3 pins"
-			(at 242.57 43.18 0)
-			(hide yes)
-			(show_name no)
-			(do_not_autoplace no)
-			(effects
-				(font
-					(size 1.27 1.27)
-				)
-			)
-		)
-		(pin "1"
-		)
-		(pin "3"
-		)
-		(pin "2"
-		)
-		(instances
-			(project "USB-Thumb-Drive"
-				(path "/61284d1f-c8a6-45b4-aa7f-ae2816ab8ea5/ca50ca8d-e0c7-4aad-ae92-c1fe4b50bba9"
-					(reference "NT602")
-					(unit 1)
-				)

Commit message: fin du schema et debut annotations precises
Parts:
- removed NT601: NetTie_3, symbol Device:NetTie_3
- added NT601, NT602: NetTie_2, symbol Device:NetTie_2
- added TP601: TestPoint, symbol Connector:TestPoint
Connections:
- net VCC: now also NT601.2, NT602.2, TP601.1
- net VCCQ: now also NT601.1
- net Vddim_eMMC: now also NT602.1
- no-connect marks 0 -> 8
Other:
- note added: "Infos choix des valeurs des composants"
- moved on the sheet: C601, C602, C603, C604, C605, C606, FB601, R601, R602, R603, R604, R605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

Commit message: fin des annotations, schema terminé
Other:
- note added: "Justification : voir infos choix composants"
- note added: "Reset"
